Commit message: diff drive controller

File: yudhaan_description/urdf/yudhaan.macro.xacro (robot description, xacro)
@@ -11,5 +11,5 @@
               <origin rpy="0 1.5707 1.5707" xyz="0 0 0"/>
               <geometry>
-                <cylinder length="0.04" radius="0.1"/>
+                <cylinder length="0.04" radius="0.05"/>
               </geometry>
             </collision>
@@ -17,5 +17,5 @@
               <origin rpy="0 1.5707 1.5707" xyz="0 0 0"/>
               <geometry>
-                <cylinder length="0.04" radius="0.1"/>
+                <cylinder length="0.04" radius="0.05"/>
               </geometry>
             </visual>
@@ -29,5 +29,4 @@
         <axis rpy="0 0 0" xyz="0 1 0"/>
         <limit effort="10000" velocity="1000"/>
-        <joint_properties damping="1.0" friction="1.0"/>
       </joint>
     </xacro:macro>

File: yudhaan_description/urdf/yudhaan.xacro (robot description, xacro)
@@ -28,5 +28,5 @@
     <!-- caster front -->
     <collision name="caster_front_collision">
-      <origin rpy=" 0 0 0" xyz="0.35 0 -0.05"/>
+      <origin rpy=" 0 0 0" xyz="0.20 -0.1 0"/>
       <geometry>
         <sphere radius="0.05"/>
@@ -44,5 +44,27 @@
     </collision>
     <visual name="caster_front_visual">
-      <origin rpy=" 0 0 0" xyz="0.2 0 -0.05"/>
+      <origin rpy=" 0 0 0" xyz="0.20 -0.1 0"/>
+      <geometry>
+        <sphere radius="0.05"/>
+      </geometry>
+    </visual>
+    <collision name="caster_front1_collision">
+      <origin rpy=" 0 0 0" xyz="0.20 0.1 0"/>
+      <geometry>
+        <sphere radius="0.05"/>
+      </geometry>
+      <surface>
+        <friction>
+          <ode>
+            <mu>0</mu>
+            <mu2>0</mu2>
+            <slip1>1.0</slip1>
+            <slip2>1.0</slip2>
+          </ode>
+        </friction>
+      </surface>
+    </collision>
+    <visual name="caster_front_visual1">
+      <origin rpy=" 0 0 0" xyz="0.20 0.1 0"/>
       <geometry>
         <sphere radius="0.05"/>
@@ -52,10 +74,9 @@
   <!-- Create wheel right -->
    <xacro:link_wheel name="link_right_wheel" />
-   <xacro:joint_wheel name="joint_right_wheel"  child="link_right_wheel"  origin_xyz="-0.05 0.15 0"  />
+   <xacro:joint_wheel name="joint_right_wheel"  child="link_right_wheel"  origin_xyz="-0.15 0.15 0"  />
   <!-- Left Wheel link -->
-  <xacro:link_wheel name="link_left_wheel" />
-  <xacro:joint_wheel name="joint_left_wheel"   child="link_left_wheel"   origin_xyz="-0.05 -0.15 0"  />
+<xacro:link_wheel name="link_left_wheel" />
+  <xacro:joint_wheel name="joint_left_wheel"   child="link_left_wheel"   origin_xyz="-0.15 -0.15 0"  />
   <link name="sensor_laser">
-    <xacro:cylinder_inertia mass="1" r="0.05" l="0.1" />
     <visual>
       <origin xyz="0 0 0" rpy="0 0 0" />
@@ -72,8 +93,28 @@
     </collision>
   </link>
-  <joint name="joint_sensor_laser" type="fixed">
-    <origin xyz="0.15 0 0.05" rpy="0 0 0"/>
+  <joint name="joint_laser_sensor" type="fixed">
+    <origin xyz="0.20 0 0.05" rpy="0 0 0"/>
     <parent link="link_chassis"/>
     <child link="sensor_laser"/>
   </joint>
+  <link name="robot_support">
+    <visual>
+      <origin xyz="0 0 0" rpy="0 0 0" />
+      <geometry>
+        <cylinder radius="0.07" length="0.1"/>
+      </geometry>
+      <material name="white" />
+    </visual>
+    <collision>
+      <origin xyz="0 0 0" rpy="0 0 0"/>
+      <geometry>
+        <cylinder radius="0.05" length="0.1"/>
+      </geometry>
+    </collision>
+  </link>
+  <joint name="joint_robot" type="fixed">
+    <origin xyz="-0.15 0 0.085" rpy="0 0 0"/>
+    <parent link="link_chassis"/>
+    <child link="robot_support"/>
+  </joint>
 </robot>
