Commit message: add world

File: yudhaan_description/urdf/yudhaan.xacro (robot description, xacro)
@@ -28,5 +28,5 @@
     <!-- caster front -->
     <collision name="caster_front_collision">
-      <origin rpy=" 0 0 0" xyz="0.20 -0.1 0"/>
+      <origin rpy=" 0 0 0" xyz="0.20 0 0"/>
       <geometry>
         <sphere radius="0.05"/>
@@ -35,8 +35,8 @@
         <friction>
           <ode>
-            <mu>0</mu>
-            <mu2>0</mu2>
-            <slip1>1.0</slip1>
-            <slip2>1.0</slip2>
+            <mu>1000000</mu>
+            <mu2>100</mu2>
+            <slip1>0.0</slip1>
+            <slip2>0.0</slip2>
           </ode>
         </friction>
@@ -44,38 +44,16 @@
     </collision>
     <visual name="caster_front_visual">
-      <origin rpy=" 0 0 0" xyz="0.20 -0.1 0"/>
+      <origin rpy=" 0 0 0" xyz="0.20 0 0"/>
       <geometry>
         <sphere radius="0.05"/>
       </geometry>
     </visual>
-    <collision name="caster_front1_collision">
-      <origin rpy=" 0 0 0" xyz="0.20 0.1 0"/>
-      <geometry>
-        <sphere radius="0.05"/>
-      </geometry>
-      <surface>
-        <friction>
-          <ode>
-            <mu>0</mu>
-            <mu2>0</mu2>
-            <slip1>1.0</slip1>
-            <slip2>1.0</slip2>
-          </ode>
-        </friction>
-      </surface>
-    </collision>
-    <visual name="caster_front_visual1">
-      <origin rpy=" 0 0 0" xyz="0.20 0.1 0"/>
-      <geometry>
-        <sphere radius="0.05"/>
-      </geometry>
-    </visual>
-    </link>
+  </link>
   <!-- Create wheel right -->
-   <xacro:link_wheel name="link_right_wheel" />
-   <xacro:joint_wheel name="joint_right_wheel"  child="link_right_wheel"  origin_xyz="-0.15 0.15 0"  />
+  <xacro:link_wheel name="link_right_wheel" />
+  <xacro:joint_wheel name="joint_right_wheel"  child="link_right_wheel"  origin_xyz="-0.05 0.15 0"  />
   <!-- Left Wheel link -->
-<xacro:link_wheel name="link_left_wheel" />
-  <xacro:joint_wheel name="joint_left_wheel"   child="link_left_wheel"   origin_xyz="-0.15 -0.15 0"  />
+  <xacro:link_wheel name="link_left_wheel" />
+  <xacro:joint_wheel name="joint_left_wheel"   child="link_left_wheel"   origin_xyz="-0.05 -0.15 0"  />
   <link name="sensor_laser">
     <visual>
