Commit message: design change

File: yudhaan_description/urdf/yudhaan.gazebo.xacro (robot description, xacro)
@@ -6,10 +6,37 @@
   <gazebo reference="link_left_wheel">
     <material>Gazebo/Blue</material>
+    <mu1>0.1</mu1>
+    <mu2>0.1</mu2>
+    <kp>1000000.0</kp>
+    <kd>10.0</kd>
+    <minDepth>0.001</minDepth>
+    <maxVel>1.0</maxVel>
+    <fdir1>0 1 0</fdir1>
   </gazebo>
   <gazebo reference="link_right_wheel">
     <material>Gazebo/Blue</material>
+    <mu1>0.1</mu1>
+    <mu2>0.1</mu2>
+    <kp>1000000.0</kp>
+    <kd>10.0</kd>
+    <minDepth>0.001</minDepth>
+    <maxVel>1.0</maxVel>
+    <fdir1>0 1 0</fdir1>
   </gazebo>
-  <gazebo reference="sensor_laser">
-    <material>Gazebo/Blue</material>
+  <gazebo reference="link_front_support">
+    <mu1>0.0</mu1>
+    <mu2>0.0</mu2>
+    <kp>1000000.0</kp>
+    <kd>100.0</kd>
+    <minDepth>0.001</minDepth>
+    <maxVel>1.0</maxVel>
+  </gazebo>
+  <gazebo reference="link_rear_support">
+    <mu1>0.0</mu1>
+    <mu2>0.0</mu2>
+    <kp>1000000.0</kp>
+    <kd>100.0</kd>
+    <minDepth>0.001</minDepth>
+    <maxVel>1.0</maxVel>
   </gazebo>
   <gazebo>
@@ -17,5 +44,28 @@
     </plugin>
   </gazebo>
+  <!-- gazebo>
+    <plugin name="gazebo_ros_control" filename="libgazebo_ros_diff_drive.so">
+      <commandTopic>cmd_vel</commandTopic>
+      <odometryTopic>odom</odometryTopic>
+      <odometryFrame>odom</odometryFrame>
+      <odometrySource>world</odometrySource>
+      <publishOdomTF>true</publishOdomTF>
+      <robotBaseFrame>link_chassis</robotBaseFrame>
+      <publishWheelTF>true</publishWheelTF>
+      <publishTf>true</publishTf>
+      <publishWheelJointState>true</publishWheelJointState>
+      <legacyMode>false</legacyMode>
+      <updateRate>30</updateRate>
+      <leftJoint>joint_left_wheel</leftJoint>
+      <rightJoint>joint_right_wheel</rightJoint>
+      <wheelSeparation>0.6</wheelSeparation>
+      <wheelDiameter>0.1</wheelDiameter>
+      <wheelAcceleration>1</wheelAcceleration>
+      <wheelTorque>10</wheelTorque>
+      <rosDebugLevel>na</rosDebugLevel>
+    </plugin>
+  </gazebo-->
   <gazebo reference="sensor_laser">
+    <material>Gazebo/Blue</material>
     <sensor type="ray" name="head_hokuyo_sensor">
       <pose>0 0 0 0 0 0</pose>

File: yudhaan_description/urdf/yudhaan.macro.xacro (robot description, xacro)
@@ -1,36 +1,33 @@
 <?xml version="1.0"?>
 <robot xmlns:xacro="http://wiki.ros.org/xacro">
-    <xacro:macro name="link_wheel" params="name">
+    <xacro:macro name="link_cyl" params="name mass r l origin_rpy origin_xyz">
         <link name="${name}">
             <inertial>
-              <mass value="2"/>
-              <origin rpy="0 1.5707 1.5707" xyz="0 0 0"/>
-              <inertia ixx="0.00526666666667" ixy="0" ixz="0" iyy="0.00526666666667" iyz="0" izz="0.01"/>
+              <mass value="${mass}"/>
+              <origin rpy="${origin_rpy}" xyz="${origin_xyz}"/>
+              <inertia ixx="${mass*(3*r*r+l*l)/12}" ixy = "0" ixz = "0" iyy="${mass*(3*r*r+l*l)/12}" iyz = "0" izz="${mass*(r*r)/2}" />
             </inertial>
-            <collision name="link_right_wheel_collision">
-              <origin rpy="0 1.5707 1.5707" xyz="0 0 0"/>
+            <collision name="${name}_collision">
+              <origin rpy="${origin_rpy}" xyz="${origin_xyz}"/>
               <geometry>
-                <cylinder length="0.04" radius="0.05"/>
+                <cylinder length="${l}" radius="${r}"/>
               </geometry>
             </collision>
             <visual name="${name}_visual">
-              <origin rpy="0 1.5707 1.5707" xyz="0 0 0"/>
+              <origin rpy="${origin_rpy}" xyz="${origin_xyz}"/>
               <geometry>
-                <cylinder length="0.04" radius="0.05"/>
+                <cylinder length="${l}" radius="${r}"/>
               </geometry>
             </visual>
         </link>
     </xacro:macro>
-    <xacro:macro name="joint_wheel" params="name child origin_xyz">
-      <joint name="${name}" type="continuous">
-        <origin rpy="0 0 0" xyz="${origin_xyz}"/>
+    <xacro:macro name="joint_cyl" params="name parent child origin_rpy origin_xyz axis_rpy axis_xyz type">
+      <joint name="${name}" type="${type}">
+        <origin rpy="${origin_rpy}" xyz="${origin_xyz}"/>
         <child link="${child}"/>
-        <parent link="link_chassis"/>
-        <axis rpy="0 0 0" xyz="0 1 0"/>
+        <parent link="${parent}"/>
+        <axis rpy="${axis_rpy}" xyz="${axis_xyz}"/>
         <limit effort="10000" velocity="1000"/>
       </joint>
     </xacro:macro>
-    <xacro:macro name="cylinder_inertia" params="mass r l">
-      <inertia ixx="${mass*(3*r*r+l*l)/12}" ixy = "0" ixz = "0" iyy="${mass*(3*r*r+l*l)/12}" iyz = "0" izz="${mass*(r*r)/2}" />
-    </xacro:macro>
 </robot>

File: yudhaan_description/urdf/yudhaan.xacro (robot description, xacro)
@@ -7,92 +7,19 @@
   <xacro:include filename="$(find yudhaan_robot)/yudhaan_description/urdf/yudhaan.transmission.xacro" />
   <!-- Chasis defined here -->
-  <link name="link_chassis">
-    <pose>0 0 0.1 0 0 0</pose>
-    <inertial>
-      <mass value="50"/>
-      <origin rpy="0 0 0" xyz="0 0 0.1"/>
-      <inertia ixx="0.395416666667" ixy="0" ixz="0" iyy="1.06208333333" iyz="0" izz="1.06208333333"/>
-    </inertial>
-    <collision name="collision_chassis">
-      <geometry>
-        <box size="0.5 0.3 0.07"/>
-      </geometry>
-    </collision>
-    <visual>
-      <origin rpy="0 0 0" xyz="0 0 0"/>
-      <geometry>
-        <box size="0.5 0.3 0.07"/>
-      </geometry>
-      <material name="blue"/>
-    </visual>
-    <!-- caster front -->
-    <collision name="caster_front_collision">
-      <origin rpy=" 0 0 0" xyz="0.20 0 0"/>
-      <geometry>
-        <sphere radius="0.05"/>
-      </geometry>
-      <surface>
-        <friction>
-          <ode>
-            <mu>1000000</mu>
-            <mu2>100</mu2>
-            <slip1>0.0</slip1>
-            <slip2>0.0</slip2>
-          </ode>
-        </friction>
-      </surface>
-    </collision>
-    <visual name="caster_front_visual">
-      <origin rpy=" 0 0 0" xyz="0.20 0 0"/>
-      <geometry>
-        <sphere radius="0.05"/>
-      </geometry>
-    </visual>
-  </link>
+  <xacro:link_cyl name="link_chassis" mass="30.0" r="0.3" l="0.1" origin_rpy="0.0 0.0 0.0" origin_xyz="0.0 0.0 0.0" />
   <!-- Create wheel right -->
-  <xacro:link_wheel name="link_right_wheel" />
-  <xacro:joint_wheel name="joint_right_wheel"  child="link_right_wheel"  origin_xyz="-0.05 0.15 0"  />
-  <!-- Left Wheel link -->
-  <xacro:link_wheel name="link_left_wheel" />
-  <xacro:joint_wheel name="joint_left_wheel"   child="link_left_wheel"   origin_xyz="-0.05 -0.15 0"  />
-  <link name="sensor_laser">
-    <visual>
-      <origin xyz="0 0 0" rpy="0 0 0" />
-      <geometry>
-        <cylinder radius="0.05" length="0.1"/>
-      </geometry>
-      <material name="white" />
-    </visual>
-    <collision>
-      <origin xyz="0 0 0" rpy="0 0 0"/>
-      <geometry>
-        <cylinder radius="0.05" length="0.1"/>
-      </geometry>
-    </collision>
-  </link>
-  <joint name="joint_laser_sensor" type="fixed">
-    <origin xyz="0.20 0 0.05" rpy="0 0 0"/>
-    <parent link="link_chassis"/>
-    <child link="sensor_laser"/>
-  </joint>
-  <link name="robot_support">
-    <visual>
-      <origin xyz="0 0 0" rpy="0 0 0" />
-      <geometry>
-        <cylinder radius="0.07" length="0.1"/>
-      </geometry>
-      <material name="white" />
-    </visual>
-    <collision>
-      <origin xyz="0 0 0" rpy="0 0 0"/>
-      <geometry>
-        <cylinder radius="0.05" length="0.1"/>
-      </geometry>
-    </collision>
-  </link>
-  <joint name="joint_robot" type="fixed">
-    <origin xyz="-0.15 0 0.085" rpy="0 0 0"/>
-    <parent link="link_chassis"/>
-    <child link="robot_support"/>
-  </joint>
+  <xacro:link_cyl name="link_right_wheel" mass="3.0" r="0.1" l="0.06"  origin_rpy="0.0 1.5707 1.5707" origin_xyz="0.0 0.0 0.0" />
+  <xacro:joint_cyl name="joint_right_wheel"  parent="link_chassis"  child="link_right_wheel"  origin_rpy="0.0 0.0 0.0"  origin_xyz="0.0 -0.3 0" axis_rpy="0 0 0" axis_xyz="0 1 0" type="continuous"/>
+  <!-- Create wheel left -->
+  <xacro:link_cyl name="link_left_wheel" mass="3.0" r="0.1" l="0.06" origin_rpy="0.0 1.5707 1.5707" origin_xyz="0.0 0.0 0.0" />
+  <xacro:joint_cyl name="joint_left_wheel"  parent="link_chassis"  child="link_left_wheel"  origin_rpy="0.0 0.0 0.0"  origin_xyz="0.0 0.3 0" axis_rpy="0 0 0" axis_xyz="0 1 0" type="continuous" />
+  <!-- Create support front -->
+  <xacro:link_cyl name="link_front_support" mass="0.0" r="0.025" l="0.05" origin_rpy="0.0 0.0 0.0" origin_xyz="0.0 0.0 0.0" />
+  <xacro:joint_cyl name="joint_front_support"  parent="link_chassis"  child="link_front_support"  origin_rpy="0.0 0.0 0.0"  origin_xyz="0.275 0.0 -0.075" axis_rpy="0 0 0" axis_xyz="0 0 0" type="fixed" />
+  <!-- Create support rear -->
+  <xacro:link_cyl name="link_rear_support" mass="0.0" r="0.025" l="0.05" origin_rpy="0.0 0.0 0.0" origin_xyz="0.0 0.0 0.0" />
+  <xacro:joint_cyl name="joint_rear_support"  parent="link_chassis"  child="link_rear_support"  origin_rpy="0.0 0.0 0.0"  origin_xyz="-0.275 0.0 -0.075" axis_rpy="0 0 0" axis_xyz="0 0 0" type="fixed" />
+  <!-- Create laser sensor -->
+  <xacro:link_cyl name="sensor_laser" mass="0.0" r="0.04" l="0.05" origin_rpy="0.0 0.0 0.0" origin_xyz="0.0 0.0 0.0" />
+  <xacro:joint_cyl name="joint_sensor_laser"  parent="link_chassis"  child="sensor_laser"  origin_rpy="0.0 0.0 0.0"  origin_xyz="0.25 0.0 0.075" axis_rpy="0 0 0" axis_xyz="0 0 0" type="fixed" />
 </robot>
